File: Telemetry peripheral boards/F3 peripheral boards.kicad_sch (KiCad schematic)
At the start: 36 parts, among them J1 ATS668LSM, J2 1053131108, J3 Potentiometer, J4 Strain Gauge, U1 LM2907M/NOPB, U2 INA125U, U3 MCP2515-I/SO, U4 ISO1050DUB

Commit message: Peripheral Boards with Attiny 1616 symbol added
Parts:
- added U5: ATTINY1616-SNR, Package_SO:SOIC-20W_7.5x12.8mm_P1.27mm, symbol New_Library:ATTINY1616-MNR
Changed lines of the file:
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@@
+	)
+	(symbol
+		(lib_id "New_Library:ATTINY1616-MNR")
+		(at 189.23 80.01 0)
+		(unit 1)
+		(exclude_from_sim no)
+		(in_bom yes)
+		(on_board yes)
+		(dnp no)
+		(fields_autoplaced yes)
+		(property "Reference" "U5"
+			(at 227.33 69.85 0)
+			(effects
+				(font
+					(size 1.524 1.524)
+				)
+			)
+		)
+		(property "Value" "ATTINY1616-SNR"
+			(at 227.33 72.39 0)
+			(effects
+				(font
+					(size 1.524 1.524)
+				)
+			)
+		)
+		(property "Footprint" "Package_SO:SOIC-20W_7.5x12.8mm_P1.27mm"
+			(at 188.976 69.85 0)
+			(effects
+				(font
+					(size 1.27 1.27)
+					(italic yes)
+				)
+				(hide yes)
+			)
+		)
+		(property "Datasheet" "ATTINY1616-MNR"
+			(at 193.548 61.468 0)
+			(effects
+				(font
+					(size 1.27 1.27)
+					(italic yes)
+				)
+				(hide yes)
+			)
+		)
+		(property "Description" ""
+			(at 189.23 80.01 0)
+			(effects
+				(font
+					(size 1.27 1.27)
+				)
+				(hide yes)
+			)
+		)
+		(pin "18"
+		)
+		(pin "8"
+		)
+		(pin "19"
+		)
+		(pin "2"
+		)
+		(pin "20"
+		)
+		(pin "17"
+		)
+		(pin "7"
+		)
+		(pin "1"
+		)
+		(pin "9"
+		)
+		(pin "6"
+		)
+		(pin "4"
+		)
+		(pin "16"
+		)
+		(pin "11"
+		)
+		(pin "14"
+		)
+		(pin "13"
+		)
+		(pin "10"
+		)
+		(pin "5"
+		)
+		(pin "12"
+		)
+		(pin "21"
+		)
+		(pin "15"
+		)
+		(pin "3"
+		)
+		(instances
+			(project ""
+				(path "/dca14ea9-6ab5-4637-ab7d-1bf40ef85725"
+					(reference "U5")
+					(unit 1)
+				)
+			)
+		)
 	)
 	(symbol
